File: PCB/MFMPico.kicad_sch (KiCad schematic)
At the start: 29 parts, among them J1 ECON34, J2 Conn_02x04_Odd_Even, J3 Micro_SD_Card, J4 Conn_01x16, J5 Conn_01x04, J6 Conn_01x02, J7 Conn_01x02, P1 CON20, U2 74LS03, U3 74LS03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

Commit message: Mostly up to date PCB
Parts:
- removed R10, R11, R6, R7, R8, R9: 1K, Resistor_SMD:R_0603_1608Metric, symbol Device:R
- removed R5: R, Resistor_SMD:R_0603_1608Metric, symbol Device:R
- added C6: 100n, Capacitor_THT:C_Disc_D3.4mm_W2.1mm_P2.50mm, symbol Device:C
- added D1: 1N5818, Diode_THT:D_DO-41_SOD81_P10.16mm_Horizontal, symbol Diode:1N5818
- added H1, H2, H3, H4, H5, H6: MountingHole, MountingHole:MountingHole_3.2mm_M3, symbol Mechanical:MountingHole
- added J8: Conn_01x02, Connector_PinHeader_2.54mm:PinHeader_1x02_P2.54mm_Vertical, symbol Connector_Generic:Conn_01x02
- added J9: Conn_01x04, Connector_PinHeader_2.54mm:PinHeader_1x04_P2.54mm_Vertical, symbol Connector_Generic:Conn_01x04
- added Q1: BC547, Package_TO_SOT_THT:TO-92_Inline, symbol Transistor_BJT:BC547
- added R12: 5.1K, Resistor_THT:R_Axial_DIN0207_L6.3mm_D2.5mm_P10.16mm_Horizontal, symbol Device:R
- added R13: 220R, Resistor_THT:R_Axial_DIN0207_L6.3mm_D2.5mm_P10.16mm_Horizontal, symbol Device:R
- added RN1, RN2: R_Network09, Resistor_THT:R_Array_SIP10, symbol Device:R_Network09
- added SW1: SW_Push, Button_Switch_THT:SW_PUSH_6mm, symbol Switch:SW_Push
- added U6: 74LS03, Package_DIP:DIP-14_W7.62mm, symbol 74xx:74LS03
- C1, C2, C3, C4, C5: footprint Capacitor_SMD:C_0603_1608Metric -> Capacitor_THT:C_Disc_D3.4mm_W2.1mm_P2.50mm
- J3: footprint Connector_Card:microSD_HC_Molex_47219-2001 -> rik:microSD Hanbo Electronic TF-018
- R2: value 5.1K -> 470R
- R3: value 1K -> 470R
- R4: value R -> 100R
Connections:
- net +3.3V: now also RN2.1 (common)
- net +5V: now also C6.1, D1.2 (A), R13.1, RN1.1 (common), U6.14 (VCC); no longer R4.1
- net DIR_IN: now also A1.16 (GPIO12), J4.12 (Pin_12), RN2.7 (R6); no longer A1.17 (GPIO13), J4.13 (Pin_13)
- net DRIVE_SEL: now also Q1.3 (E), R13.2, U6.2, U6.5; no longer J2.1 (Pin_1), J2.3 (Pin_3), J2.5 (Pin_5), J2.7 (Pin_7), J7.1 (Pin_1)
- net GND: now also C6.2, Q1.1 (C), SW1.1, U6.7 (GND)
- net HEAD_0: now also A1.17 (GPIO13), J4.13 (Pin_13), RN2.8 (R7); no longer A1.19 (GPIO14), J4.14 (Pin_14)
- net HEAD_1: now also RN2.5 (R4)
- net HEAD_2: now also A1.19 (GPIO14), J4.14 (Pin_14), RN2.9 (R8); no longer A1.20 (GPIO15), J4.15 (Pin_15)
- net MFM_IN: now also U5.2 (RO); no longer R2.2, U5.3 (RE), U5.4 (DE)
- net MFM_OUT: no longer U5.2 (RO)
- net STEP: now also A1.15 (GPIO11), J4.11 (Pin_11), RN2.6 (R5); no longer A1.16 (GPIO12), J4.12 (Pin_12)
- net WRITE_GATE: now also RN2.4 (R3); no longer R3.2
- net ~WRITE_GATE: now reaches J1.6 (Write_gate), U4.5
- net ~WRITE_GATE: now also RN1.5 (R4), U6.4
- net HEAD_3: now reaches U2.6
- net HEAD_3: now also A1.20 (GPIO15), J4.15 (Pin_15), RN2.10 (R9); no longer P1.1 (Drive_Selected)
- net at P1.13 (MFM_Write+), R1.1, U5.12 (RI_A): now also J9.1 (Pin_1)
- net at P1.14 (MFM_Write-), R1.2, U5.11 (RI_B): now also J9.2 (Pin_2)
- net at P1.17 (MFM_Read+), U5.9 (DO_Y): now also R4.2, J9.4 (Pin_4)
- net at P1.18 (MFM_Read-), U5.10 (DO_Z): now also R4.1, J9.3 (Pin_3)
- net at A1.30 (RUN): now also SW1.2
- net at A1.39 (VSYS): now also D1.1 (K); no longer R4.2
- net at J1.4 (Head_2), U4.10: now also RN1.4 (R3)
- net at J1.24 (Step), U2.2: now also RN1.8 (R7)
- net at J1.34 (Direction_In), U4.13: now also RN1.10 (R9)
- net at J1.14 (Head_0), U3.5: now also RN1.6 (R5)
- net at J1.18 (Head_1), U3.2: now also RN1.7 (R6)
- net at J1.2 (Head_3/REDWR): now also U2.5, RN1.3 (R2)
- removed net SELECT: A1.15 (GPIO11), J4.11 (Pin_11), J7.2 (Pin_2), U2.5
- new net: J7.1 (Pin_1), U6.1, U6.6
- new net: J8.1 (Pin_1), U6.3
- new net: J7.2 (Pin_2), R2.2, U5.4 (DE)
- new net: J8.2 (Pin_2), R3.2, U5.3 (RE)
- new net: Q1.2 (B), R12.1
- new net ~DRIVE_SEL: J2.1 (Pin_1), J2.3 (Pin_3), J2.5 (Pin_5), J2.7 (Pin_7), P1.1 (Drive_Selected), R12.2, RN1.9 (R8)
- no-connect marks 18 -> 27
Other:
- moved on the sheet: J1, J2, U2A, U2B, U2C, U2D, U3A, U3B, U3C, U3D, U4A, U4B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
